File: Wifi_WX_Station/Base.sch (EAGLE design)
At the start: 62 parts, among them IC1 25LC512, IC2 3.3v, IC3 PIC24FJ128GA008, Q2 32Khz, X1 MINI-USB-VERT

Commit message: added all the small boards, renamed Wifi module as RH and LH version
Parts:
- removed ANA_IN: (no value), con-lsta:FE06-1
- removed BHT: MA1X06, wifi_WX:MA1X06
- removed I2C2: (no value), SparkFun-Connectors:M03PTH
- removed IC2: 3.3v, Stofer:78MXXL
- removed JP2: M05X2SHD, wifi_WX:M05X2SHD
- removed LED1, LED2, LED3, LED4, LED5: (no value), led:LEDCHIP-LED0603
- removed X1: MINI-USB-VERT, wifi_WX:MINI-USB-VERT
- added ANA: (no value), SparkFun-Connectors:M04PTH
- added C19, C20, C21: 0.1uF, rcl:C-USC0805
- added I2C1: (no value), wifi_WX:PINHD-1X3
- added J5: MA1X06, wifi_WX:MA1X06
- added J6: M05X22X5FE, wifi_WX:M05X22X5FE
- added L1: grn, led:LEDCHIP-LED0603
- added L2: ambr, led:LEDCHIP-LED0603
- added L3: red, led:LEDCHIP-LED0603
- added R2: 120o, rcl:R-US_R0603
- added R21, R22: 26.1K, rcl:R-US_R0603
- added R4: 10k, rcl:R-US_R0603
- added RESET: SWITCH-MOMENTARY-2SMD, SparkFun-Electromechanical:SWITCH-MOMENTARY-2SMD
- added TP1, TP2: TPTP06R, 1AA_Stofer:TPTP06R
- added TP3: TPTP10R, 1AA_Stofer:TPTP10R
- added U2: 25LC512, microchip:25LC080SN
- added USB: MINI-USB-32005-301, wifi_WX:MINI-USB-32005-301
- C1: value 22p -> 22u/10v; device rcl:C-USC0603 -> rcl:CPOL-USSMCB
- C10, C9: value 0.1u -> 2.2uF
- C11: value 2.2u -> 0.1uF; device rcl:C-USC1206 -> rcl:C-USC0805
- C12: value 2.2u -> 22uF/10V; device rcl:C-USC1206 -> rcl:CPOL-USSMCB
- C13: value 0.1uf -> 0.1uF
- C14: value 1u -> 22p; device rcl:C-USC0805 -> rcl:C-USC0603
- C15: value 10uf/6v -> 22p; device rcl:CPOL-USSMCA -> rcl:C-USC0603
- C16, C17, C18, C3, C4, C5: value 0.1u -> 0.1uF
- C2: value 22p -> 0.1uF; device rcl:C-USC0603 -> rcl:C-USC0805
- C6: value 4.7u -> 0.1uF; device rcl:C-USC1210 -> rcl:C-USC0805
- C7: value 22u/10v -> 330uF/6V; device rcl:CPOL-USR/2012-12R -> rcl:CPOL-USSMCD
- C8: value 100u/4v -> 0.1uF; device rcl:CPOL-USR/2012-12R -> rcl:C-USC0805
- FAN, SUN, UART1: device SparkFun-Connectors:M03PTH -> wifi_WX:PINHD-1X3
- IC1: value 25LC512 -> 3.3v; device microchip:25LC080SN -> Stofer:78MXXL
- R1: value 120 -> 120o
- R10: value 14k -> 26.1K
- R11: value 26.4K -> 10k
- R12: value 4.7k -> 4.7K
- R13: value 120 -> 4.7k
- R14: value 10k -> 4.7K
- R15: value 1k -> 4.7k
- R18: value 120 -> 470o
- R19, R20: value 1k -> 14k
- R5: value 10k -> 8.2k
- R6: value 10k -> 26.1k
- R7: value 6.8k -> 14k
- R8: value 26.4K -> 14k
- R9: value 4.7k -> 26.1K
- SV1, SV3: device con-lsta:FE10-1 -> wifi_WX:FE10-1
- SV2: device con-lsta:FE10-1 -> wifi_WX:FE10-1; OC_FARNELL (none) -> unknown; OC_NEWARK (none) -> unknown
- renumbered IC3 to U3, JP1 to JPROG, Q2 to Q1, U$1 to U1, U$3 to J1
Connections:
- removed net N$43: ANA_IN.5, U3.PGD1/EMUD1/AN0/CN2/RB0
- removed net N$46: LED4.A, R19.1
- removed net N$64: ANA_IN.4, U3.PGC1/EMUC1/AN1/CN3/RB1
- removed net N$65: ANA_IN.3, U3.C2IN-/AN2/SS1/CN4/RB2
- removed net N$67: LED5.A, R20.1
- removed net N$68: LED4.C, U1.GPIO.0
- removed net N$69: LED5.C, U1.GPIO.1
- new net N$14: TP2.TP, U3.OSC1/CLKI/RC12
- new net N$18: L3.A, R16.2
- new net N$20: L2.A, R17.2
- new net N$21: L1.A, R18.2
- new net N$4: TP1.TP, U3.OSC2/CLKO/RC15
- new net N$5: R18.1, U3.PMD5/RE5
- net +3V3: now also C11.2, C18.1, C19.2, C6.1, C7.+, C8.1, IC1.VO, J5.6, J6.10, R11.1, R12.1, R13.2, R14.1, R15.2, U2.!HOLD, U2.!WP, U2.VCC; no longer ANA_IN.1, BHT.6, C3.1, C5.1, C8.+, C9.1, IC1.!HOLD, IC1.!WP, IC1.VCC, IC2.VO, JP2.10, R12.2, R19.2, R20.2, R3.1, R9.2
- net +5V: now also C1.+, C2.1, FAN.1, IC1.VI, R3.1; no longer C10.1, C7.+, IC2.VI, R5.1
- net BARO_CS: now also J5.2; no longer BHT.2
- net GND: now also ANA.1, C1.-, C12.-, C15.2, C20.2, C21.2, C8.2, FAN.3, I2C1.2, J5.1, J6.2, L1.C, L2.C, L3.C, R10.1, R21.1, R22.1, R4.1, R9.1, RESET.2, RESET.3, S1.4, S2.4, U2.GND, USB.5_GND, USB.SHLD; no longer ANA_IN.6, BHT.1, C1.2, C11.2, C12.2, C15.-, C8.-, I2C2.2, IC2.GND, JP2.2, R11.1, R15.2, R16.2, R17.2, R8.1, X1.5_GND
- net MCU_RESET_: now also JPROG.VPP_MCLR, R11.2, RESET.1, RESET.4; no longer R13.2, R14.2
- net MRF_CS_: now also J6.5; no longer JP2.5
- net MRF_HIBER: now also J6.3; no longer JP2.3
- net MRF_RESET_: now also J6.4; no longer JP2.4
- net MRF_SCK: now also J6.8; no longer JP2.8
- net MRF_SDI: now also J6.9; no longer JP2.9
- net MRF_SDO: now also J6.6; no longer JP2.6
- net N$1: now also I2C1.1; no longer I2C2.1
- net N$19: now also C12.+; no longer C15.+
- net N$2: now also C15.1; no longer BHT.5, C1.1
- net N$22: now also C21.1, R7.2, R9.2, U3.PGD1/EMUD1/AN0/CN2/RB0; no longer C14.1, R14.1, R3.2
- net N$23: now also ANA.4, R20.1; no longer LED1.C, R17.1
- net N$24: now also C20.1, R19.2, R21.2, U3.PGC1/EMUC1/AN1/CN3/RB1; no longer JPROG.VPP_MCLR, R13.1
- net N$25: now also U2.SO; no longer IC1.SO
- net N$27: now also U2.!CS; no longer IC1.!CS
- net N$28: now also C3.1, R20.2, R22.2, U3.C2IN-/AN2/SS1/CN4/RB2; no longer LED2.C, R16.1
- net N$29: now also U2.SCK; no longer IC1.SCK
- net N$3: now also C10.1; no longer C6.1, U1.VPP
- net N$30: now also ANA.3, R19.1; no longer LED3.C, R15.1
- net N$31: now also ANA.2, R7.1; no longer LED1.A, U3.PMD5/RE5
- net N$32: now also U2.SI; no longer IC1.SI
- net N$33: now also R17.1; no longer LED2.A
- net N$34: now also R16.1; no longer LED3.A
- net N$37: now also S2.3
- net N$38: now also S1.3
- net N$6: now also I2C1.3; no longer I2C2.3
- net N$66: now also C5.1, R3.2, R4.2; no longer C18.1, R5.2, R6.2
- net N$7: now also C14.1; no longer C2.1
- net N$8: now also TP3.TP, U3.TDO/INT2/RE9; no longer ANA_IN.2, U3.T4CK/RC3
- net N$9: now also USB.1_VBUS; no longer X1.1_VBUS
- net RAIN_CNT_IN: now also R2.1; no longer R18.1
- net RAIN_COUNT: now also C11.1, R15.1, R2.2, U3.T4CK/RC3; no longer R12.1, R18.2, U3.TDO/INT2/RE9
- net SCL1: now also J5.4, R12.2; no longer BHT.4
- net SDA1: now also J5.3, R14.2; no longer BHT.3
- net SUN_ADC_IN: now also R8.2; no longer C12.1, R11.2
- net SUN_IN: now also R8.1; no longer R10.1
- net USB_D+: now also USB.3_D+; no longer X1.3_D+
- net USB_D-: now also USB.2_D-; no longer X1.2_D-
- net WIFI_INT_: now also J6.7; no longer JP2.7
- net WIND_ADC_IN: now also C9.1, R5.2, R6.2; no longer C11.1, R7.2, R8.2
- net WIND_COUNT: now also C19.1, R13.1; no longer R9.1
- net WIN_DIR_IN: now also R5.1; no longer R7.1
Other:
- note added: "R19 and R20 not loaded"
- note added: "calc TC"
- note removed: "Female"
- moved on the sheet: C10, C11, C13, C14, C16, C17, C18, C2, C3, C4, C5, C6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

Commit message: updated BOM with all prices- As Checked in to BATCH PCB
Parts:
- removed C17: 0.1uF, rcl:C-USC0805
- added R23, R24: 4.7K, rcl:R-US_R0603
- ANA: device SparkFun-Connectors:M04PTH -> wifi_WX:M04PTH
- FAN, SUN: device wifi_WX:PINHD-1X3 -> wifi_WX:PINHD-1X3MOLEX_KK
- IC1: device Stofer:78MXXL -> wifi_WX:78MXXL
- J5: value MA1X06 -> (none); device wifi_WX:MA1X06 -> wifi_WX:M05MOLEX_KK
- Q1: value 32Khz -> 32.768Khz; device crystal:CRYSTALTC26V -> wifi_WX:CRYSTAL
- RESET, S1, S2: device SparkFun-Electromechanical:SWITCH-MOMENTARY-2SMD -> wifi_WX:SWITCH-MOMENTARY-2SMD
- SV1: value (none) -> M10"; device wifi_WX:FE10-1 -> wifi_WX:M10"
- SV2, SV3: value (none) -> M10"; device wifi_WX:FE10-1 -> wifi_WX:M10"; OC_FARNELL unknown -> (none); OC_NEWARK unknown -> (none)
- TP1, TP2: value TPTP06R -> TP; device 1AA_Stofer:TPTP06R -> wifi_WX:TP
- TP3: value TPTP10R -> TP; device 1AA_Stofer:TPTP10R -> wifi_WX:TP
Connections:
- removed net N$1: I2C1.1, U3.SCL2/INT3/RA14
- removed net N$3: C10.1
- removed net N$6: I2C1.3, U3.SDA2/INT4/RA15
- new net SCL2: I2C1.1, R24.2, U3.SCL2/INT3/RA14
- new net SDA2: I2C1.3, R23.2, U3.SDA2/INT4/RA15
- net +3V3: now also J5.5, R23.1, R24.1; no longer C17.1, J5.6
- net GND: no longer C17.2
- net N$14: now also TP3.P$1; no longer TP2.TP
- net N$2: now also Q1.P$2; no longer Q1.2
- net N$4: now also TP2.P$1; no longer TP1.TP
- net N$7: now also Q1.P$1; no longer Q1.1
- net N$8: now also TP1.P$1; no longer TP3.TP
- net SUN_ADC_IN: now also C10.1
Other:
- moved on the sheet: C15, C16, C18, I2C1, J6, R10, R12, R14, SV1, SV2, SV3, UART1

Commit message: Wind speed board and base station rework to rev HW 1.2
Parts:
- added +5V: (no value), wifi_WX:PINHD-1X3MOLEX_KK
- added D2: MBR0520LT, diode:MBR0520LT
- added RAIN: M02, wifi_WX:M02
- ANA: device wifi_WX:M04PTH -> wifi_WX:M05PTH
- R13: value 4.7k -> 2.2K
- TP1: value TP -> TP10R; device wifi_WX:TP -> wifi_WX:TP10R
- TP2, TP3: value TP -> TP6R; device wifi_WX:TP -> wifi_WX:TP6R
Connections:
- new net N$1: D2.C, R2.2
- net +5V: now also +5V.1, ANA.5
- net GND: now also +5V.3, RAIN.1
- net RAIN_CNT_IN: now also RAIN.2
- net RAIN_COUNT: now also D2.A; no longer R2.2
Other:
- moved on the sheet: FAN, TP1, TP2, TP3
Changed lines of the file:
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@@
 <part name="R6" library="rcl" deviceset="R-US_" device="R0603" value="26.1k"/>
 <part name="C9" library="rcl" deviceset="C-US" device="C0805" value="2.2uF"/>
-<part name="R13" library="rcl" deviceset="R-US_" device="R0603" value="4.7k"/>
+<part name="R13" library="rcl" deviceset="R-US_" device="R0603" value="2.2K"/>
 <part name="R3" library="rcl" deviceset="R-US_" device="R0603" value="10k"/>
 <part name="C10" library="rcl" deviceset="C-US" device="C0805" value="2.2uF"/>
@@
 <part name="C20" library="rcl" deviceset="C-US" device="C0805" value="0.1uF"/>
 <part name="C21" library="rcl" deviceset="C-US" device="C0805" value="0.1uF"/>
-<part name="ANA" library="wifi_WX" deviceset="M04" device="PTH"/>
 <part name="J5" library="wifi_WX" deviceset="M05" device="MOLEX_KK"/>
 <part name="SUPPLY13" library="supply2" deviceset="GND" device=""/>
 <part name="R23" library="rcl" deviceset="R-US_" device="R0603" value="4.7K"/>
 <part name="R24" library="rcl" deviceset="R-US_" device="R0603" value="4.7K"/>
-<part name="TP1" library="wifi_WX" deviceset="TP" device=""/>
-<part name="TP2" library="wifi_WX" deviceset="TP" device=""/>
-<part name="TP3" library="wifi_WX" deviceset="TP" device=""/>
+<part name="TP1" library="wifi_WX" deviceset="TP" device="10R" value="TP10R"/>
+<part name="TP2" library="wifi_WX" deviceset="TP" device="6R"/>
+<part name="TP3" library="wifi_WX" deviceset="TP" device="6R"/>
 <part name="Q1" library="wifi_WX" deviceset="CRYSTAL" device="" value="32.768Khz"/>
+<part name="RAIN" library="wifi_WX" deviceset="M02" device=""/>
+<part name="SUPPLY10" library="supply2" deviceset="GND" device=""/>
+<part name="+5V" library="wifi_WX" deviceset="PINHD-1X3" device="MOLEX_KK"/>
+<part name="ANA" library="wifi_WX" deviceset="M05" device="PTH"/>
+<part name="P+4" library="supply1" deviceset="+5V" device=""/>
+<part name="D2" library="diode" deviceset="MBR0520LT" device=""/>
 </parts>
 <sheets>
@@
 <instance part="UART1" gate="A" x="-10.16" y="-2.54" rot="R270"/>
 <instance part="I2C1" gate="A" x="93.98" y="50.8"/>
-<instance part="FAN" gate="A" x="-243.84" y="-33.02"/>
+<instance part="FAN" gate="A" x="-254" y="-33.02"/>
 <instance part="SUN" gate="A" x="-243.84" y="-15.24"/>
 <instance part="SV1" gate="G$1" x="-66.04" y="-43.18" rot="MR90"/>
@@
 </instance>
 <instance part="R7" gate="G$1" x="-198.12" y="22.86" smashed="yes">
-<attribute name="NAME" x="-201.93" y="26.8986" size="1.778" layer="95"/>
-<attribute name="VALUE" x="-196.088" y="26.924" size="1.778" layer="96"/>
+<attribute name="NAME" x="-201.93" y="24.3586" size="1.778" layer="95"/>
+<attribute name="VALUE" x="-193.548" y="24.384" size="1.778" layer="96"/>
 </instance>
 <instance part="R9" gate="G$1" x="-193.04" y="12.7" rot="R90"/>
 <instance part="R19" gate="G$1" x="-198.12" y="27.94" smashed="yes">
-<attribute name="NAME" x="-201.93" y="31.9786" size="1.778" layer="95"/>
-<attribute name="VALUE" x="-196.088" y="32.004" size="1.778" layer="96"/>
+<attribute name="NAME" x="-204.47" y="29.4386" size="1.778" layer="95"/>
+<attribute name="VALUE" x="-193.548" y="29.464" size="1.778" layer="96"/>
 </instance>
 <instance part="R20" gate="G$1" x="-198.12" y="33.02" smashed="yes">
-<attribute name="NAME" x="-201.93" y="37.0586" size="1.778" layer="95"/>
-<attribute name="VALUE" x="-196.088" y="37.084" size="1.778" layer="96"/>
+<attribute name="NAME" x="-204.47" y="34.5186" size="1.778" layer="95"/>
+<attribute name="VALUE" x="-193.548" y="34.544" size="1.778" layer="96"/>
 </instance>
 <instance part="R21" gate="G$1" x="-185.42" y="12.7" rot="R90"/>
@@
 <instance part="C20" gate="G$1" x="-160.02" y="12.7"/>
 <instance part="C21" gate="G$1" x="-152.4" y="12.7"/>
-<instance part="ANA" gate="G$1" x="-215.9" y="25.4"/>
 <instance part="J5" gate="G$1" x="116.84" y="48.26" rot="MR0"/>
 <instance part="SUPPLY13" gate="GND" x="81.28" y="50.8" smashed="yes" rot="R270"/>
@@
 </instance>
 <instance part="Q1" gate="Q$1" x="7.62" y="78.74"/>
+<instance part="RAIN" gate="G$1" x="-279.4" y="22.86"/>
+<instance part="SUPPLY10" gate="GND" x="-266.7" y="12.7"/>
+<instance part="+5V" gate="A" x="-276.86" y="-33.02"/>
+<instance part="ANA" gate="G$1" x="-218.44" y="27.94"/>
+<instance part="P+4" gate="1" x="-210.82" y="35.56" smashed="yes">
+<attribute name="VALUE" x="-210.82" y="35.56" size="1.778" layer="96" rot="R90"/>
+</instance>
+<instance part="D2" gate="G$1" x="-233.68" y="33.02" rot="R270"/>
 </instances>
 <busses>
@@
 <pinref part="SUPPLY11" gate="GND" pin="GND"/>
 <wire x1="-264.16" y1="-38.1" x2="-264.16" y2="-35.56" width="0.1524" layer="91"/>
-<wire x1="-264.16" y1="-35.56" x2="-246.38" y2="-35.56" width="0.1524" layer="91"/>
+<wire x1="-264.16" y1="-35.56" x2="-256.54" y2="-35.56" width="0.1524" layer="91"/>
 <pinref part="FAN" gate="A" pin="3"/>
+<pinref part="+5V" gate="A" pin="3"/>
+<wire x1="-279.4" y1="-35.56" x2="-264.16" y2="-35.56" width="0.1524" layer="91"/>
 </segment>
 <segment>
@@
 <pinref part="J5" gate="G$1" pin="1"/>
 <wire x1="109.22" y1="43.18" x2="109.22" y2="35.56" width="0.1524" layer="91"/>
+</segment>
+<segment>
+<wire x1="-266.7" y1="20.32" x2="-266.7" y2="15.24" width="0.1524" layer="91"/>
+<pinref part="SUPPLY10" gate="GND" pin="GND"/>
+<pinref part="RAIN" gate="G$1" pin="1"/>
+<wire x1="-269.24" y1="20.32" x2="-266.7" y2="20.32" width="0.1524" layer="91"/>
 </segment>
 </net>
@@
 <pinref part="P+3" gate="1" pin="+5V"/>
 <wire x1="-264.16" y1="-27.94" x2="-264.16" y2="-30.48" width="0.1524" layer="91"/>
-<wire x1="-264.16" y1="-30.48" x2="-246.38" y2="-30.48" width="0.1524" layer="91"/>
+<wire x1="-264.16" y1="-30.48" x2="-256.54" y2="-30.48" width="0.1524" layer="91"/>
 <pinref part="FAN" gate="A" pin="1"/>
+<pinref part="+5V" gate="A" pin="1"/>
+<wire x1="-279.4" y1="-30.48" x2="-264.16" y2="-30.48" width="0.1524" layer="91"/>
+</segment>
+<segment>
+<pinref part="ANA" gate="G$1" pin="5"/>
+<pinref part="P+4" gate="1" pin="+5V"/>
 </segment>
 </net>
@@
 <segment>
 <pinref part="R15" gate="G$1" pin="1"/>
-<pinref part="R2" gate="G$1" pin="2"/>
 <wire x1="-152.4" y1="40.64" x2="-152.4" y2="63.5" width="0.1524" layer="91"/>
 <wire x1="-152.4" y1="63.5" x2="-152.4" y2="91.44" width="0.1524" layer="91"/>
-<wire x1="-241.3" y1="0" x2="-236.22" y2="0" width="0.1524" layer="91"/>
-<wire x1="-236.22" y1="0" x2="-236.22" y2="40.64" width="0.1524" layer="91"/>
-<wire x1="-236.22" y1="40.64" x2="-215.9" y2="40.64" width="0.1524" layer="91"/>
 <pinref part="U3" gate="G$1" pin="T4CK/RC3"/>
 <junction x="-152.4" y="63.5"/>
@@
 <pinref part="C11" gate="G$1" pin="1"/>
 <wire x1="-215.9" y1="45.72" x2="-215.9" y2="40.64" width="0.1524" layer="91"/>
+<pinref part="D2" gate="G$1" pin="A"/>
+<wire x1="-233.68" y1="35.56" x2="-233.68" y2="40.64" width="0.1524" layer="91"/>
+<wire x1="-233.68" y1="40.64" x2="-215.9" y2="40.64" width="0.1524" layer="91"/>
 </segment>
 </net>
@@
 <segment>
 <label x="-281.94" y="0" size="0.8128" layer="95" rot="R180" xref="yes"/>
+<pinref part="J1" gate="G$1" pin="7"/>
+<wire x1="-261.62" y1="0" x2="-264.16" y2="0" width="0.1524" layer="91"/>
+<wire x1="-261.62" y1="22.86" x2="-261.62" y2="0" width="0.1524" layer="91"/>
+<pinref part="RAIN" gate="G$1" pin="2"/>
+<wire x1="-269.24" y1="22.86" x2="-261.62" y2="22.86" width="0.1524" layer="91"/>
 <pinref part="R2" gate="G$1" pin="1"/>
-<wire x1="-251.46" y1="0" x2="-264.16" y2="0" width="0.1524" layer="91"/>
-<pinref part="J1" gate="G$1" pin="7"/>
+<wire x1="-261.62" y1="0" x2="-251.46" y2="0" width="0.1524" layer="91"/>
 </segment>
 </net>
@@
 <segment>
 <pinref part="U3" gate="G$1" pin="OSC1/CLKI/RC12"/>
-<wire x1="-12.7" y1="45.72" x2="5.08" y2="45.72" width="0.1524" layer="91"/>
+<wire x1="-12.7" y1="45.72" x2="0" y2="45.72" width="0.1524" layer="91"/>
 <pinref part="TP3" gate="G$1" pin="P$1"/>
 </segment>
@@
 <segment>
 <pinref part="U3" gate="G$1" pin="OSC2/CLKO/RC15"/>
-<wire x1="-12.7" y1="48.26" x2="-3.81" y2="48.26" width="0.1524" layer="91"/>
+<wire x1="-12.7" y1="48.26" x2="-8.89" y2="48.26" width="0.1524" layer="91"/>
 <pinref part="TP2" gate="G$1" pin="P$1"/>
 </segment>
@@
 <pinref part="U3" gate="G$1" pin="TDO/INT2/RE9"/>
 <pinref part="TP1" gate="G$1" pin="P$1"/>
-<wire x1="-142.24" y1="40.64" x2="-134.62" y2="40.64" width="0.1524" layer="91"/>
+<wire x1="-137.16" y1="40.64" x2="-134.62" y2="40.64" width="0.1524" layer="91"/>
 </segment>
 </net>
@@
 </segment>
 </net>
+<net name="N$1" class="0">
+<segment>
+<pinref part="R2" gate="G$1" pin="2"/>
+<pinref part="D2" gate="G$1" pin="C"/>
+<wire x1="-241.3" y1="0" x2="-233.68" y2="0" width="0.1524" layer="91"/>
+<wire x1="-233.68" y1="0" x2="-233.68" y2="30.48" width="0.1524" layer="91"/>
+</segment>
+</net>

Commit message: Revision B.1
Parts:
- C5: value 0.1uF -> 2.2uF
Connections:
- removed net N$37: S2.2, S2.3, U3.!U1RTS/BCLK1/CN21/RD15
- removed net N$38: S1.2, S1.3, U3.!U1CTS/CN20/RD14
- new net SW_S1: S1.2, S1.3, U1.GPIO.1, U3.!U1CTS/CN20/RD14
- new net SW_S2: S2.2, S2.3, U1.GPIO.2, U3.!U1RTS/BCLK1/CN21/RD15
- net MCU_RESET_: now also U1.GPIO.0
Other:
- note added: "MRF24"
- note removed: "R19 and R20 not loaded"
- note removed: "calc TC"
- moved on the sheet: C11, C14, C15, C19, R15
