File: Wifi_WX_Station/Wind_enc.sch (EAGLE design)
At the start: 11 parts, among them U1 AS5030

Commit message: Added multiple new boards - H-pwrdist- Insp_Wind_enc, 5040 etc..
Other:
- note added: "B.1"
- note removed: "B.2"
Changed lines of the file:
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@@
 <text x="-30.48" y="66.04" size="1.778" layer="91">GND</text>
 <text x="119.38" y="-12.7" size="3.81" layer="94" ratio="20">WunderWxStation</text>
-<text x="181.61" y="-34.036" size="3.81" layer="94" ratio="20">B.2</text>
+<text x="181.61" y="-34.036" size="3.81" layer="94" ratio="20">B.1</text>
 </plain>
 <instances>
