File: NanoModemAX25/NanoModem.brd (EAGLE design)
At the start: 43.5 x 25.4 mm, 49 parts, among them IC1 FT232RL, Q1 T2N7002AK, X1 MINI-USB-32005-201, Y1 16MHz

Commit message: some changes to the APRS modem board
Parts:
- added C4: 1uF, rcl:C0603
- added R17: 1k, rcl:R0603
- C8: device rcl:C0805 -> rcl:C1210
- R12: value 10 -> 330
- R6: value 1k -> 10k
- moved R11 3.98 mm to (18.3, 10.5)
- moved C3 2.29 mm to (17.8, 6.99)
- moved R10 2.29 mm to (15.9, 6.99)
- moved R12 2.29 mm to (19.7, 6.99)
- moved C8 0.90 mm to (13.3, 9.53)
Connections:
- removed net N$9: C2.1, R5.1, R5.2
- new net A_REF: 328P.20, C4.2, R11.2, R17.2
- new net N$11: C2.1, R5.1
- net 3V3: now also R17.1; no longer 328P.20, 3V3.1, R11.2
- net ANALOG_OUT: now also R5.2
- net GND: now also C4.1
Routing:
- net 3V3: track 33.9 -> 15.2 mm, vias 1 -> 0
- net A_REF: track 0.00 -> 8.78 mm
- net N$9: track 8.52 -> 0.00 mm
- net N$11: track 0.00 -> 7.94 mm
- net GND: track 154.4 -> 158.7 mm
- net FTDI_TX: track 13.4 -> 17.4 mm
- net ANALOG_OUT: track 8.30 -> 11.0 mm
- net 5V: track 78.1 -> 79.8 mm
- net MCU_RX: track 15.7 -> 17.1 mm, vias 2 -> 1
- net ADC0: track 10.6 -> 9.25 mm
- net RESET: track 50.8 -> 49.6 mm
- net ANALOG_IN: track 5.39 -> 4.45 mm
- net MOSI: track 4.67 -> 3.96 mm
